File: MCU data logger.kicad_sch (KiCad schematic)
At the start: 0 parts

Commit message: Complete hierarchical schematic design for MCU Data Logger
Parts:
- added 100nF1, C4: 100nF, symbol Device:C
- added BT1: Battery, symbol Device:Battery
- added C1: 0.1uF, symbol Device:C
- added C2, C3: 22pF, symbol Device:C
- added D1, D2: LED, symbol Device:LED
- added R1, R2, R6: 10k, symbol Device:R
- added R3, R4: 4.7k, symbol Device:R
- added R5, R7: 330, symbol Device:R
- added U1: ATMEGA328P-AN, ATMEGA328P-AN:QFP80P900X900X120-32N, symbol ATMEGA328P-AN:ATMEGA328P-AN
- added U2: DS1337S_, DS1337S_:SOIC127P600X175-8N, symbol DS1337S_:DS1337S_
- added U3, U4: 24LC1025, symbol Memory_EEPROM:24LC1025
- added Y1: 32.768Khz, symbol Device:Crystal
- added Y2: 16MHz, symbol Device:Crystal
Connections:
- new net: R2.2, U2.7 (SQW/~INT)
- new net: U2.2 (X2), Y1.1
- new net: U2.1 (X1), Y1.2
- new net: D1.1 (K), R5.2
- new net: D2.1 (K), R7.1
- new net: R1.2, U2.3 (~{INTA})
- new net: C4.2, U1.20 (AREF)
- new net: C3.2, U1.8 (PB7), Y2.1
- new net: C2.2, U1.7 (PB6), Y2.2
- new net D2: U1.32 (PD2)
- new net D3: U1.1 (PD3)
- new net D4: U1.2 (PD4)
- new net D5: U1.9 (PD5)
- new net D6: U1.10 (PD6)
- new net D7: U1.11 (PD7)
- new net D8: U1.12 (PB0)
- new net GND: 100nF1.2, BT1.2 (-), C1.2, C2.1, C3.1, C4.1, R5.1, R7.2, U1.21 (GND), U1.3 (GND), U1.5 (GND), U2.4 (GND), U3.4 (GND), U3.7 (WP), U4.2 (A1), U4.4 (GND), U4.7 (WP)
- new net MISO: U1.16 (PB4)
- new net MOSI: U1.15 (PB3)
- new net RESET: R6.2, U1.29 (PC6/~{RESET})
- new net RX: U1.30 (PD0)
- new net TX: U1.31 (PD1)
- new net VCC: 100nF1.1, BT1.1 (+), C1.1, D2.2 (A), R1.1, R2.1, R3.1, R4.1, R6.1, U1.18 (AVCC), U1.4 (VCC), U1.6 (VCC), U2.8 (VCC), U3.1 (A0), U3.2 (A1), U3.3 (A2), U3.8 (VCC), U4.1 (A0), U4.3 (A2), U4.8 (VCC)
- new net sck: D1.2 (A), R3.2, U1.17 (PB5), U1.28 (PC5), U2.6 (SCL), U3.6 (SCL), U4.6 (SCL)
- new net sda: R4.2, U1.27 (PC4), U2.5 (SDA), U3.5 (SDA), U4.5 (SDA)
- no-connect marks 0 -> 8
Other:
- added sheet connectors (connectors.kicad_sch)
- note added: "EEPROM"
- note added: "Real Time Clock"
- company: (none) -> chis
- title: (none) -> MCU DATA LOGGER
