File: _restore_backup_2026-07-03T21-34-06-555/MCU data logger.kicad_sch (KiCad schematic)
At the start: 25 parts, among them U1 ATMEGA328P-AN, U2 DS1337S_, U3 24LC1025, U4 24LC1025, Y1 32.768Khz, Y2 16MHz

Commit message: Completed 2-layer PCB layout
Parts:
- removed H1, H2, H3, H4: MountingHole, MountingHole:MountingHole_2.1mm, symbol Mechanical:MountingHole
- 100nF1: renamed from C5; footprint Capacitor_SMD:C_0805_2012Metric -> (none)
- BT1: footprint Connector_PinHeader_2.54mm:PinHeader_1x02_P2.54mm_Vertical -> (none)
- C1, C2, C3: footprint Capacitor_SMD:C_0805_2012Metric -> (none)
- C4: value 0.1uF -> 100nF; footprint Capacitor_SMD:C_0805_2012Metric -> (none)
- D1, D2: footprint LED_SMD:LED_0805_2012Metric -> (none)
- R1, R2, R3, R4, R5, R6, R7: footprint Resistor_SMD:R_0805_2012Metric -> (none)
- U3, U4: footprint Package_SO:SOIC-8_5.3x5.3mm_P1.27mm -> (none)
- Y1, Y2: footprint Crystal:Crystal_SMD_5032-2Pin_5.0x3.2mm_HandSoldering -> (none)
